Commit message: finish nmpc

File: src/models/inverted_pendulum/cartpole.urdf (robot description, URDF)
Before this commit: robot cartpole, 3 links, 2 joints
Links:
- link cart: geometry collision box size=0.1 0.1 0.1; visual box size=0.5 0.5 0.2
- link pole: geometry collision cylinder size=0.05 1.0; visual cylinder size=0.05 1.0
